File: Project Net Class/Project Net Class.kicad_sch (KiCad schematic)
At the start: 7 parts

Commit message: 계층 구조 테스트
계층 구조 테스트
실제 PCB는 언제 짜볼라나
Other:
- added sheet Sheet_2 (sheet_2.kicad_sch)
Changed lines of the file:
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@@
 	(generator_version "9.0")
 	(paper "A4")
+	(junction
+		(at 190.5 66.04)
+		(diameter 0)
+		(color 0 0 0 0)
+	)
 	(wire
 		(pts
@@
 	(wire
 		(pts
+			(xy 190.5 104.14) (xy 190.5 66.04)
+		)
+		(stroke
+			(width 0)
+			(type default)
+		)
+	)
+	(wire
+		(pts
 			(xy 176.53 46.99) (xy 190.5 46.99)
 		)
@@
 	(wire
 		(pts
+			(xy 147.32 104.14) (xy 190.5 104.14)
+		)
+		(stroke
+			(width 0)
+			(type default)
+		)
+	)
+	(wire
+		(pts
 			(xy 190.5 66.04) (xy 175.26 66.04)
 		)
@@
 	(wire
 		(pts
-			(xy 175.26 73.66) (xy 144.78 73.66)
+			(xy 144.78 73.66) (xy 175.26 73.66)
 		)
 		(stroke
@@
 				)
 			)
+		)
+	)
+	(sheet
+		(at 53.34 93.98)
+		(size 93.98 54.61)
+		(exclude_from_sim no)
+		(in_bom yes)
+		(on_board yes)
+		(dnp no)
+		(fields_autoplaced yes)
+		(stroke
+			(width 0.1524)
+			(type solid)
+		)
+		(fill
+			(color 0 0 0 0.0000)
+		)
+		(property "Sheetname" "Sheet_2"
+			(at 53.34 93.2684 0)
+			(effects
+				(font
+					(size 1.27 1.27)
+				)
+				(justify left bottom)
+			)
+		)
+		(property "Sheetfile" "sheet_2.kicad_sch"
+			(at 53.34 149.1746 0)
+			(effects
+				(font
+					(size 1.27 1.27)
+				)
+				(justify left top)
+			)
+		)
+		(pin "H_1_Label" output
+			(at 147.32 104.14 0)
+			(effects
+				(font
+					(size 1.27 1.27)
+				)
+				(justify right)
+			)
+		)
+		(instances
+			(project "Project Net Class"
+				(path "/105f2309-8062-4052-83a1-4f56df5cd5b0"
+					(page "2")
+				)
+			)
