File: Project Net Class/Project Net Class.kicad_pcb (KiCad board)
At the start: 2 copper layers, 7 parts

Commit message: 망했다
뭐가 빠졌을라나
Parts:
- added R1000: R, Resistor_SMD:R_0201_0603Metric, F.Cu at (161.2, 74.2)
- added R122: R, Resistor_SMD:R_0201_0603Metric, F.Cu at (164.7, 78.5)
- added R8: R, Resistor_SMD:R_0201_0603Metric, F.Cu at (145.7, 80.2)
- added R9: R, Resistor_SMD:R_0201_0603Metric, F.Cu at (153.5, 87.2)
- moved R4 10.6 mm to (103.3, 106.2), turned to 180 degrees
- moved R7 4.94 mm to (108.5, 103.2), turned to 90 degrees
- moved R3 4.66 mm to (105.2, 102.5), turned to -90 degrees
